File: shield/shield.kicad_pcb (KiCad board)
At the start: 2 copper layers, 68.6 x 53.3 mm, 58 parts, among them U1 CD4051B

Commit message: Release 8x6 arduino shield rev 1
Other:
- board text added: "ὀπτικός 8x6 arduino shield https://github.com/majkrzak/optikos Date: 2022-01-02 Rev: 1"
Changed lines of the file:
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@@
   )
   (paper "A5")
+  (title_block
+    (title "ὀπτικός 8x6 arduino shield")
+    (date "2022-01-02")
+    (rev "1")
+    (company "Piotr Majkrzak")
+  )
   (layers
     (0 "F.Cu" signal)
@@
     (effects (font (size 2.5 2.5) (thickness 0.5)))
   )
+  (gr_text "ὀπτικός 8x6 arduino shield\nhttps://github.com/majkrzak/optikos\nDate: 2022-01-02 Rev: 1" (at 123.825 81.28) (layer "F.SilkS")
+    (effects (font (size 0.5 0.5) (thickness 0.125)) (justify left))
+  )
   (segment (start 80.645 39.37) (end 88.265 39.37) (width 0.2286) (layer "B.Cu") (net 3))
