File: shield/shield.kicad_sch (KiCad schematic)
At the start: 58 parts, among them U1 CD4051B

Commit message: Release 8x6 arduino shield rev 1
Other:
- company: (none) -> Piotr Majkrzak
- title: (none) -> ὀπτικός 8x6 arduino shield
Changed lines of the file:
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@@
 (kicad_sch (version 20211123) (generator eeschema)
   (paper "A4")
+  (title_block
+    (title "ὀπτικός 8x6 arduino shield")
+    (date "2022-01-02")
+    (rev "1")
+    (company "Piotr Majkrzak")
+  )
   (junction (at 215.9 106.68) (diameter 0) (color 0 0 0 0)
   )
